Commit message: Imported upstream version '0.5.6' of 'upstream'

File: share/urdf/nao.urdf (robot description, URDF)
Before this commit: robot naoH25V50, 79 links, 78 joints
Links:
- added link MicroFrontCenter_frame
- added link MicroRearCenter_frame
- added link MicroSurroundLeft_frame
- added link MicroSurroundRight_frame
- link LFsrFL_frame: mass None -> 2e-06; geometry collision box size=0.01 0.01 0.005
- link LFsrFR_frame: mass None -> 2e-06; geometry collision box size=0.01 0.01 0.005
- link LFsrRL_frame: mass None -> 2e-06; geometry collision box size=0.01 0.01 0.005
- link LFsrRR_frame: mass None -> 2e-06; geometry collision box size=0.01 0.01 0.005
- link LHip: mass 0.14053 -> 0.13053
- link LShoulder: mass 0.09304 -> 0.07504
- link LTibia: mass 0.30142 -> 0.29142
- link Neck: mass 0.07842 -> 0.06442
- link RFsrFL_frame: mass None -> 2e-06; geometry collision box size=0.01 0.01 0.005
- link RFsrFR_frame: mass None -> 2e-06; geometry collision box size=0.01 0.01 0.005
- link RFsrRL_frame: mass None -> 2e-06; geometry collision box size=0.01 0.01 0.005
- link RFsrRR_frame: mass None -> 2e-06; geometry collision box size=0.01 0.01 0.005
- link RHip: mass 0.14053 -> 0.13053
- link RShoulder: mass 0.09304 -> 0.07504
- link RTibia: mass 0.30142 -> 0.29142
- link l_ankle: mass 0.17184 -> 0.16184
- link r_ankle: mass 0.17184 -> 0.16184
Joints:
- removed joint CameraBottom_optical_frame_joint
- removed joint CameraTop_optical_frame_joint
- added joint CameraBottom_optical_frame_fixedjoint: type fixed, parent CameraBottom_frame, child CameraBottom_optical_frame, origin xyz=0 0 0 rpy=-1.57079632679 0 -1.57079632679
- added joint CameraTop_optical_frame_fixedjoint: type fixed, parent CameraTop_frame, child CameraTop_optical_frame, origin xyz=0 0 0 rpy=-1.57079632679 0 -1.57079632679
- added joint MicroFront_sensor_fixedjoint: type fixed, parent Head, child MicroFrontCenter_frame, origin xyz=0.041 0 0.091 rpy=0 0 0, axis 0 0 0
- added joint MicroLeft_sensor_fixedjoint: type fixed, parent Head, child MicroSurroundLeft_frame, origin xyz=-0.0195 0.0606 0.0331 rpy=0 0 0, axis 0 0 0
- added joint MicroRear_sensor_fixedjoint: type fixed, parent Head, child MicroRearCenter_frame, origin xyz=-0.0577 0 0.0693 rpy=0 0 0, axis 0 0 0
- added joint MicroRight_sensor_fixedjoint: type fixed, parent Head, child MicroSurroundRight_frame, origin xyz=-0.0195 -0.0606 0.0331 rpy=0 0 0, axis 0 0 0

File: share/urdf/romeo.urdf (robot description, URDF)
Before this commit: robot romeoH37, 92 links, 91 joints
Links:
- added link CameraLeftEye_optical_frame
- added link CameraLeft_optical_frame
- added link CameraRightEye_optical_frame
- added link CameraRight_optical_frame
- link HeadPitch_link: mass 0.13728 -> 0.158407
- link HeadRoll_link: mass 1.79432 -> 2.07047
- link LAnklePitch_link: mass 0.42803 -> 0.464512
- link LElbow: mass 0.36997 -> 0.460203
- link LFinger11_link: mass None -> 2e-06
- link LFinger12_link: mass None -> 2e-06
- link LFinger13_link: mass None -> 2e-06
- link LFinger21_link: mass None -> 2e-06
- link LFinger22_link: mass None -> 2e-06
- link LFinger23_link: mass None -> 2e-06
- link LFinger31_link: mass None -> 2e-06
- link LFinger32_link: mass None -> 2e-06
- link LFinger33_link: mass None -> 2e-06
- link LForeArm: mass 0.48271 -> 0.600439
- link LFsrFToeFrontLeft_frame: mass None -> 2e-06; geometry collision box size=0.01 0.01 0.005
- link LFsrFToeFrontRight_frame: mass None -> 2e-06; geometry collision box size=0.01 0.01 0.005
- link LFsrFToeRearLeft_frame: mass None -> 2e-06; geometry collision box size=0.01 0.01 0.005
- link LFsrFToeRearRight_frame: mass None -> 2e-06; geometry collision box size=0.01 0.01 0.005
- link LFsrFrontCenter_frame: mass None -> 2e-06; geometry collision box size=0.01 0.01 0.005
- link LFsrHeelLeft_frame: mass None -> 2e-06; geometry collision box size=0.01 0.01 0.005
- link LFsrHeelRight_frame: mass None -> 2e-06; geometry collision box size=0.01 0.01 0.005
- link LFsrRearCenter_frame: mass None -> 2e-06; geometry collision box size=0.01 0.01 0.005
- link LHip: mass 0.65864 -> 0.714778
- link LHipYaw_link: mass 0.51527 -> 0.559188
- link LShoulder: mass 0.43527 -> 0.541429
- link LShoulderYaw_link: mass 0.69262 -> 0.861545
- link LThigh: mass 4.34097 -> 4.71096
- link LThumb1_link: mass None -> 2e-06
- link LThumb2_link: mass None -> 2e-06
- link LThumb3_link: mass None -> 2e-06
- link LTibia: mass 2.50906 -> 2.72291
- link LWristRoll_link: mass 0.17551 -> 0.218316
- link LWristYaw_link: mass 0.061 -> 0.0758774
- link NeckPitch_link: mass 0.29923 -> 0.345282
- link NeckYaw_link: mass 0.32745 -> 0.377845
- link RAnklePitch_link: mass 0.42803 -> 0.464512
- link RElbow: mass 0.36997 -> 0.460203
- link RFinger11_link: mass None -> 2e-06
- link RFinger12_link: mass None -> 2e-06
- link RFinger13_link: mass None -> 2e-06
- link RFinger21_link: mass None -> 2e-06
- link RFinger22_link: mass None -> 2e-06
- link RFinger23_link: mass None -> 2e-06
- link RFinger31_link: mass None -> 2e-06
- link RFinger32_link: mass None -> 2e-06
- link RFinger33_link: mass None -> 2e-06
- link RForeArm: mass 0.48271 -> 0.600439
- link RFsrFToeFrontLeft_frame: mass None -> 2e-06; geometry collision box size=0.01 0.01 0.005
- link RFsrFToeFrontRight_frame: mass None -> 2e-06; geometry collision box size=0.01 0.01 0.005
- link RFsrFToeRearLeft_frame: mass None -> 2e-06; geometry collision box size=0.01 0.01 0.005
- link RFsrFToeRearRight_frame: mass None -> 2e-06; geometry collision box size=0.01 0.01 0.005
- link RFsrFrontCenter_frame: mass None -> 2e-06; geometry collision box size=0.01 0.01 0.005
- link RFsrHeelLeft_frame: mass None -> 2e-06; geometry collision box size=0.01 0.01 0.005
- link RFsrHeelRight_frame: mass None -> 2e-06; geometry collision box size=0.01 0.01 0.005
- link RFsrRearCenter_frame: mass None -> 2e-06; geometry collision box size=0.01 0.01 0.005
- link RHip: mass 0.65864 -> 0.714778
- link RHipYaw_link: mass 0.51527 -> 0.559188
- link RShoulder: mass 0.43527 -> 0.541429
- link RShoulderYaw_link: mass 0.69262 -> 0.861545
- link RThigh: mass 4.34097 -> 4.71096
- link RThumb1_link: mass None -> 2e-06
- link RThumb2_link: mass None -> 2e-06
- link RThumb3_link: mass None -> 2e-06
- link RTibia: mass 2.50906 -> 2.72291
- link RWristRoll_link: mass 0.17551 -> 0.218316
- link RWristYaw_link: mass 0.061 -> 0.0758774
- link body: mass 4.4142 -> 5.11337
- link l_ankle: mass 0.98379 -> 1.06764
- link l_gripper: mass None -> 2e-06
- link l_wrist: mass 0.35549 -> 0.442191
- link r_ankle: mass 0.98379 -> 1.06764
- link r_gripper: mass None -> 2e-06
- link r_wrist: mass 0.35549 -> 0.442191
- link torso: mass 5.0541 -> 5.85463
Joints:
- added joint CameraLeftEye_optical_frame_fixedjoint: type fixed, parent CameraLeftEye_frame, child CameraLeftEye_optical_frame, origin xyz=0 0 0 rpy=-1.57079632679 0 -1.57079632679
- added joint CameraLeft_optical_frame_fixedjoint: type fixed, parent CameraLeft_frame, child CameraLeft_optical_frame, origin xyz=0 0 0 rpy=-1.57079632679 0 -1.57079632679
- added joint CameraRightEye_optical_frame_fixedjoint: type fixed, parent CameraRightEye_frame, child CameraRightEye_optical_frame, origin xyz=0 0 0 rpy=-1.57079632679 0 -1.57079632679
- added joint CameraRight_optical_frame_fixedjoint: type fixed, parent CameraRight_frame, child CameraRight_optical_frame, origin xyz=0 0 0 rpy=-1.57079632679 0 -1.57079632679
- joint HeadRoll: limit lower=-0.4887 upper=0.4887 effort=0.9 velocity=1.5 -> lower=-0.4887 upper=0.4887 effort=3.748 velocity=1.5
- joint NeckPitch: limit lower=-0.3142 upper=0.6632 effort=2.978 velocity=2.2 -> lower=-0.3142 upper=0.6632 effort=5.956 velocity=2.2
- joint NeckYaw: limit lower=-2.0595 upper=2.0595 effort=3.662 velocity=4.0 -> lower=-2.0595 upper=2.0595 effort=7.324 velocity=4.0
- joint TrunkYaw: limit lower=-0.7575 upper=0.7575 effort=80.902 velocity=1.5 -> lower=-0.7575 upper=0.7575 effort=28.021 velocity=1.5
